Commit message: 对 /gpu-train --sim梳理了框架并修复录制残留问题, 更新 sim 录制链路与自动化配置
- 调整 play_z1_video、mujoco_manual 与 orchestrator 相关逻辑
- 更新 5-phase plan、奖励配置与机器人资源

Co-Authored-By: Claude Opus 4.6 (1M context) <noreply@anthropic.com>

File: source/magiclab_rl_lab/magiclab_rl_lab/data/robots/magicbot-Z1/urdf/MagicBotZ1_23dof.urdf (robot description, URDF)
Before this commit: robot MagicBotZ1, 31 links, 30 joints
Links:
- link left_hand_palm_link: geometry collision sphere radius=0.04
- link right_hand_palm_link: geometry collision sphere radius=0.04
